File: Piprogrammer.kicad_pcb (KiCad board)
At the start: 2 copper layers, 56 x 65 mm, 27 parts, among them J1 Conn_02x01, J10 Conn_01x01, J11 QWIIC_CONNECTORJS-1MM, J2 Conn_02x01, J3 Conn_01x20, J4 Conn_01x20, J6 Conn_01x01, J7 Conn_ARM_JTAG_SWD_10, J9 Conn_01x02, P1 Conn_02x20_Odd_Even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

Commit message: minor update em schematics presentation, update to kicad 6
Other:
- net class Default removed
- net class Power removed
